File: CoRoMotorDrivers.kicad_sch (KiCad schematic)
At the start: 17 parts, among them J1 Conn_01x05, M1 Conn_01x02, M2 Conn_01x02, M3 Conn_01x02, P1 Conn_01x02, U1 L293D, U2 L293D

Commit message: Add files via upload
Connections:
- net at U2.2 (1A): now also A1.13 (D10); no longer A1.25 (A6)
- net at U2.7 (2A): now also A1.14 (MOSI); no longer A1.26 (A7)
Changed lines of the file:
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@@
   (junction (at 160.02 162.56) (diameter 0) (color 0 0 0 0)
   )
-  (junction (at 85.09 113.03) (diameter 0) (color 0 0 0 0)
-  )
   (junction (at 157.48 97.79) (diameter 0) (color 0 0 0 0)
   )
@@
   (junction (at 222.25 162.56) (diameter 0) (color 0 0 0 0)
   )
+  (junction (at 85.09 118.11) (diameter 0) (color 0 0 0 0)
+  )
   (junction (at 149.86 162.56) (diameter 0) (color 0 0 0 0)
   )
@@
     (stroke (width 0) (type default) (color 0 0 0 0))
   )
-  (wire (pts (xy 121.92 96.52) (xy 121.92 120.65))
-    (stroke (width 0) (type default) (color 0 0 0 0))
-  )
   (wire (pts (xy 46.99 63.5) (xy 55.88 63.5))
     (stroke (width 0) (type default) (color 0 0 0 0))
   )
-  (wire (pts (xy 116.84 99.06) (xy 116.84 125.73))
-    (stroke (width 0) (type default) (color 0 0 0 0))
-  )
   (wire (pts (xy 232.41 137.16) (xy 233.68 137.16))
     (stroke (width 0) (type default) (color 0 0 0 0))
@@
     (stroke (width 0) (type default) (color 0 0 0 0))
   )
+  (wire (pts (xy 121.92 115.57) (xy 121.92 120.65))
+    (stroke (width 0) (type default) (color 0 0 0 0))
+  )
   (wire (pts (xy 232.41 135.89) (xy 232.41 137.16))
     (stroke (width 0) (type default) (color 0 0 0 0))
@@
     (stroke (width 0) (type default) (color 0 0 0 0))
   )
+  (wire (pts (xy 68.58 93.98) (xy 68.58 111.76))
+    (stroke (width 0) (type default) (color 0 0 0 0))
+  )
   (wire (pts (xy 167.64 120.65) (xy 170.18 120.65))
     (stroke (width 0) (type default) (color 0 0 0 0))
@@
     (stroke (width 0) (type default) (color 0 0 0 0))
   )
-  (wire (pts (xy 85.09 106.68) (xy 85.09 113.03))
+  (wire (pts (xy 85.09 106.68) (xy 85.09 118.11))
     (stroke (width 0) (type default) (color 0 0 0 0))
   )
@@
     (stroke (width 0) (type default) (color 0 0 0 0))
   )
-  (wire (pts (xy 85.09 113.03) (xy 58.42 113.03))
+  (wire (pts (xy 85.09 118.11) (xy 58.42 118.11))
     (stroke (width 0) (type default) (color 0 0 0 0))
   )
@@
     (stroke (width 0) (type default) (color 0 0 0 0))
   )
-  (wire (pts (xy 97.79 96.52) (xy 121.92 96.52))
-    (stroke (width 0) (type default) (color 0 0 0 0))
-  )
   (wire (pts (xy 157.48 110.49) (xy 157.48 97.79))
     (stroke (width 0) (type default) (color 0 0 0 0))
@@
     (stroke (width 0) (type default) (color 0 0 0 0))
   )
-  (wire (pts (xy 97.79 99.06) (xy 116.84 99.06))
-    (stroke (width 0) (type default) (color 0 0 0 0))
-  )
   (wire (pts (xy 214.63 97.79) (xy 219.71 97.79))
     (stroke (width 0) (type default) (color 0 0 0 0))
@@
     (stroke (width 0) (type default) (color 0 0 0 0))
   )
+  (wire (pts (xy 63.5 88.9) (xy 63.5 115.57))
+    (stroke (width 0) (type default) (color 0 0 0 0))
+  )
   (wire (pts (xy 157.48 97.79) (xy 187.96 97.79))
     (stroke (width 0) (type default) (color 0 0 0 0))
@@
     (stroke (width 0) (type default) (color 0 0 0 0))
   )
+  (wire (pts (xy 72.39 93.98) (xy 68.58 93.98))
+    (stroke (width 0) (type default) (color 0 0 0 0))
+  )
   (wire (pts (xy 121.92 46.99) (xy 121.92 93.98))
     (stroke (width 0) (type default) (color 0 0 0 0))
@@
     (stroke (width 0) (type default) (color 0 0 0 0))
   )
+  (wire (pts (xy 63.5 115.57) (xy 121.92 115.57))
+    (stroke (width 0) (type default) (color 0 0 0 0))
+  )
   (wire (pts (xy 200.66 83.82) (xy 97.79 83.82))
     (stroke (width 0) (type default) (color 0 0 0 0))
@@
     (stroke (width 0) (type default) (color 0 0 0 0))
   )
+  (wire (pts (xy 72.39 88.9) (xy 63.5 88.9))
+    (stroke (width 0) (type default) (color 0 0 0 0))
+  )
   (wire (pts (xy 142.24 146.05) (xy 124.46 146.05))
     (stroke (width 0) (type default) (color 0 0 0 0))
@@
     (stroke (width 0) (type default) (color 0 0 0 0))
   )
+  (wire (pts (xy 116.84 111.76) (xy 116.84 125.73))
+    (stroke (width 0) (type default) (color 0 0 0 0))
+  )
   (wire (pts (xy 229.87 135.89) (xy 232.41 135.89))
     (stroke (width 0) (type default) (color 0 0 0 0))
   )
-  (wire (pts (xy 85.09 113.03) (xy 85.09 162.56))
-    (stroke (width 0) (type default) (color 0 0 0 0))
-  )
   (wire (pts (xy 121.92 120.65) (xy 142.24 120.65))
     (stroke (width 0) (type default) (color 0 0 0 0))
@@
     (stroke (width 0) (type default) (color 0 0 0 0))
   )
+  (wire (pts (xy 58.42 118.11) (xy 58.42 113.03))
+    (stroke (width 0) (type default) (color 0 0 0 0))
+  )
   (wire (pts (xy 187.96 130.81) (xy 187.96 97.79))
     (stroke (width 0) (type default) (color 0 0 0 0))
@@
     (stroke (width 0) (type default) (color 0 0 0 0))
   )
+  (wire (pts (xy 68.58 111.76) (xy 116.84 111.76))
+    (stroke (width 0) (type default) (color 0 0 0 0))
+  )
   (wire (pts (xy 170.18 125.73) (xy 170.18 124.46))
     (stroke (width 0) (type default) (color 0 0 0 0))
   )
+  (wire (pts (xy 85.09 118.11) (xy 85.09 162.56))
+    (stroke (width 0) (type default) (color 0 0 0 0))
+  )
