File: CoroMotorDriversDefaultDrillSize.kicad_pcb (KiCad board)
At the start: 2 copper layers, 73.7 x 68.6 mm, 17 parts, among them J1 Conn_01x05, M1 Conn_01x02, M2 Conn_01x02, M3 Conn_01x02, P1 Conn_01x02, U1 L293D, U2 L293D

Commit message: Add files via upload
Routing:
- net Net-(A1-Pad27): track 151.0 -> 196.2 mm
- net Net-(U2-Pad2): track 89.6 -> 53.0 mm
- net Net-(A1-Pad29): track 128.9 -> 163.0 mm
- net Net-(U2-Pad7): track 67.4 -> 79.4 mm
- net Net-(A1-Pad23): track 27.3 -> 18.5 mm
- net Net-(A1-Pad21): track 25.8 -> 32.9 mm
- net Net-(M2-Pad1): track 16.2 -> 21.2 mm
- net Net-(A1-Pad24): track 17.3 -> 13.0 mm
- net Net-(M1-Pad1): track 27.4 -> 25.9 mm
- net Net-(A1-Pad30): track 33.6 -> 35.1 mm
- net Net-(M2-Pad2): track 25.1 -> 23.7 mm
- net Net-(A1-Pad20): track 17.7 -> 19.1 mm
- net Net-(A1-Pad22): track 20.1 -> 19.2 mm
